File: kicad/isense.sch (KiCad schematic (older format))
At the start: 8 parts, among them U401 OPA237NA_250, U402 OPA237NA_250

Commit message: Fixes in schematics (only) done during initial debug
Parts:
- added C401: 10uF, Capacitors_Tantalum_SMD:CP_Tantalum_Case-B_EIA-3528-21_Hand, symbol Device:CP
- U401, U402: symbol OPA237NA_250:OPA237NA_250 -> st12-rescue:OPA237NA_250-OPA237NA_250
Connections:
- net GND: now also C401.2
- net I_SENSE: now also C401.1
Changed lines of the file:
@@
 $EndDescr
 $Comp
-L OPA237NA_250:OPA237NA_250 U401
+L st12-rescue:OPA237NA_250-OPA237NA_250 U401
 U 1 1 60BE946A
 P 3450 2300
@@
 $EndComp
 $Comp
-L OPA237NA_250:OPA237NA_250 U402
+L st12-rescue:OPA237NA_250-OPA237NA_250 U402
 U 1 1 60BE9D2E
 P 6600 2300
@@
 	6700 3100 7450 3100
 Wire Wire Line
-	7450 3100 7450 2200
+	7450 3100 7450 2350
 Connection ~ 7450 2200
 Wire Wire Line
@@
 Wire Wire Line
 	5300 1200 5700 1200
+$Comp
+L Device:CP C401
+U 1 1 60CA4B23
+P 8050 2700
+F 0 "C401" H 8168 2746 50  0000 L CNN
+F 1 "10uF" H 8168 2655 50  0000 L CNN
+F 2 "Capacitors_Tantalum_SMD:CP_Tantalum_Case-B_EIA-3528-21_Hand" H 8088 2550 50  0001 C CNN
+F 3 "~" H 8050 2700 50  0001 C CNN
+	1    8050 2700
+	1    0    0    -1
+$EndComp
+Wire Wire Line
+	8050 2550 8050 2350
+Wire Wire Line
+	8050 2350 7450 2350
+Connection ~ 7450 2350
+Wire Wire Line
+	7450 2350 7450 2200
+$Comp
+L power:GND #PWR0408
+U 1 1 60CA7409
+P 8050 2850
+F 0 "#PWR0408" H 8050 2600 50  0001 C CNN
+F 1 "GND" H 8055 2677 50  0000 C CNN
+F 2 "" H 8050 2850 50  0001 C CNN
+F 3 "" H 8050 2850 50  0001 C CNN
+	1    8050 2850
+	1    0    0    -1
+$EndComp
 $EndSCHEMATC

Commit message: Various schematic fixes
Parts:
- added U?: OPA237NA_250, OPA237NA:SOT95P280X145-5N, symbol st12-rescue:OPA237NA_250-OPA237NA_250
Connections:
- net +5V: now also U?.5 (V+)
- net GND: now also U?.2 (V-)
- net I_SENSE_RAW: now also U?.3 (+IN); no longer R404.2
- new net: R404.2, U?.1 (OUT), U?.4 (-IN)
Other:
- moved on the sheet: C401, R401, R402, R403, R404, R405, R406, U401, U402
