File: kicad/power.sch (KiCad schematic (older format))
At the start: 54 parts, among them J201 Conn_01x02_Male, J202 T12_Sense, J203 T12_POWER, Q201 2N7002, Q202 FDS4435BZ, U201 ACS756xCB-050B-PFF, U202 TPS5430DDAR, U203 AMS1117-5.0, U204 OPA237NA_250, U205 AMS1117-3.3

Commit message: Fixes in schematics (only) done during initial debug
Parts:
- removed R210: 7.5K, Resistors_SMD:R_0805_HandSoldering, symbol Device:R
- added C213: 100nF, Capacitors_SMD:C_1210_HandSoldering, symbol Device:C
- added C214: 470nF, Capacitors_SMD:C_2220_HandSoldering, symbol Device:C
- C208: value 220uF 6V -> 220uF 10V
- Q202: symbol FDS4435BZ:FDS4435BZ -> st12-rescue:FDS4435BZ-FDS4435BZ
- R211: value 7.5K -> 120K
- U202: symbol TPS5430DDAR:TPS5430DDAR -> st12-rescue:TPS5430DDAR-TPS5430DDAR
- U204: symbol OPA237NA_250:OPA237NA_250 -> st12-rescue:OPA237NA_250-OPA237NA_250
Connections:
- net COLD is gone; now on net COLD_SENSE: J202.4 (Pin_4)
- net GND: now also C213.2, C214.2
- net V24HEATER: now also C213.1, C214.1
Other:
- note removed: "Not sure if needed.\nDraws HEATER line up\nwhen it is unengaged"
Changed lines of the file:
@@
 $EndDescr
 $Comp
-L TPS5430DDAR:TPS5430DDAR U?
+L st12-rescue:TPS5430DDAR-TPS5430DDAR U?
 U 1 1 60B0AF4B
 P 4400 1700
@@
 AR Path="/60AEC464/60B0AFBE" Ref="C208"  Part="1"
 F 0 "C208" H 6568 1696 50  0000 L CNN
-F 1 "220uF 6V" V 6600 1250 50  0000 L CNN
+F 1 "220uF 10V" V 6600 1250 50  0000 L CNN
 F 2 "Capacitors_Tantalum_SMD:CP_Tantalum_Case-X_EIA-7343-43_Hand" H 6488 1500 50  0001 C CNN
 F 3 "~" H 6450 1650 50  0001 C CNN
@@
 Connection ~ 1950 3550
 $Comp
-L FDS4435BZ:FDS4435BZ Q?
+L st12-rescue:FDS4435BZ-FDS4435BZ Q?
 U 1 1 60B0B08F
 P 2250 4400
@@
 V24HEATER
 $Comp
-L OPA237NA_250:OPA237NA_250 U?
+L st12-rescue:OPA237NA_250-OPA237NA_250 U?
 U 1 1 60B0B126
 P 9150 3200
@@
 Wire Wire Line
 	3100 6800 3100 6750
-Text Label 2700 7100 2    50   ~ 0
+Text Label 3000 7100 2    50   ~ 0
 COLD
 Connection ~ 3100 7100
@@
 AR Path="/60AEC464/60B0B114" Ref="R211"  Part="1"
 F 0 "R211" H 3030 6904 50  0000 R CNN
-F 1 "7.5K" V 3100 7050 50  0000 R CNN
+F 1 "120K" V 3100 7050 50  0000 R CNN
 F 2 "Resistors_SMD:R_0805_HandSoldering" V 3030 6950 50  0001 C CNN
 F 3 "~" H 3100 6950 50  0001 C CNN
 	1    3100 6950
 	1    0    0    -1
-$EndComp
-$Comp
-L Device:R R?
-U 1 1 60B0B10E
-P 2850 7100
-AR Path="/60B0B10E" Ref="R?"  Part="1"
-AR Path="/60AEC464/60B0B10E" Ref="R210"  Part="1"
-F 0 "R210" H 2780 7054 50  0000 R CNN
-F 1 "7.5K" V 2850 7200 50  0000 R CNN
-F 2 "Resistors_SMD:R_0805_HandSoldering" V 2780 7100 50  0001 C CNN
-F 3 "~" H 2850 7100 50  0001 C CNN
-	1    2850 7100
-	0    -1   -1   0
 $EndComp
 $Comp
@@
 Wire Wire Line
 	850  6950 1200 6950
-Wire Notes Line
-	2750 4650 3350 4650
-Wire Notes Line
-	3350 4650 3350 5200
-Wire Notes Line
-	3350 5200 2750 5200
-Wire Notes Line
-	2750 5200 2750 4650
-Text Notes 3050 5150 0    50   ~ 0
-Not sure if needed.\nDraws HEATER line up\nwhen it is unengaged
 Wire Wire Line
 	2350 3200 2950 3200
@@
 Wire Wire Line
 	2950 3200 3150 3200
+Wire Wire Line
+	4450 3950 4900 3950
+Text Label 4450 3950 0    50   ~ 0
+V24HEATER
+$Comp
+L Device:C C?
+U 1 1 60C98FC3
+P 4900 4100
+AR Path="/60C98FC3" Ref="C?"  Part="1"
+AR Path="/60AEC464/60C98FC3" Ref="C213"  Part="1"
+F 0 "C213" H 5015 4146 50  0000 L CNN
+F 1 "100nF" H 5015 4055 50  0000 L CNN
+F 2 "Capacitors_SMD:C_1210_HandSoldering" H 4938 3950 50  0001 C CNN
+F 3 "~" H 4900 4100 50  0001 C CNN
+	1    4900 4100
+	1    0    0    -1
+$EndComp
+$Comp
+L power:GND #PWR?
+U 1 1 60C994D9
+P 4900 4250
+AR Path="/60C994D9" Ref="#PWR?"  Part="1"
+AR Path="/60AEC464/60C994D9" Ref="#PWR0239"  Part="1"
+F 0 "#PWR0239" H 4900 4000 50  0001 C CNN
+F 1 "GND" H 4905 4077 50  0000 C CNN
+F 2 "" H 4900 4250 50  0001 C CNN
+F 3 "" H 4900 4250 50  0001 C CNN
+	1    4900 4250
+	1    0    0    -1
+$EndComp
+$Comp
+L Device:C C?
+U 1 1 60C99945
+P 5450 4100
+AR Path="/60C99945" Ref="C?"  Part="1"
+AR Path="/60AEC464/60C99945" Ref="C214"  Part="1"
+F 0 "C214" H 5565 4146 50  0000 L CNN
+F 1 "470nF" H 5565 4055 50  0000 L CNN
+F 2 "Capacitors_SMD:C_2220_HandSoldering" H 5488 3950 50  0001 C CNN
+F 3 "~" H 5450 4100 50  0001 C CNN
+	1    5450 4100
+	1    0    0    -1
+$EndComp
+Wire Wire Line
+	5450 3950 4900 3950
+Connection ~ 4900 3950
+$Comp
+L power:GND #PWR?
+U 1 1 60C9F39C
+P 5450 4250
+AR Path="/60C9F39C" Ref="#PWR?"  Part="1"
+AR Path="/60AEC464/60C9F39C" Ref="#PWR0240"  Part="1"
+F 0 "#PWR0240" H 5450 4000 50  0001 C CNN
+F 1 "GND" H 5455 4077 50  0000 C CNN
+F 2 "" H 5450 4250 50  0001 C CNN
+F 3 "" H 5450 4250 50  0001 C CNN
+	1    5450 4250
+	1    0    0    -1
+$EndComp
 $EndSCHEMATC

Commit message: Various schematic fixes
Connections:
- net SHAKE is gone; now on net SHAKE_SENSE: J202.3 (Pin_3), R208.1
- net GND: now also R208.2
- net SHAKE_SENSE: no longer R208.2
Other:
- moved on the sheet: R208
Changed lines of the file:
@@
 	1    0    0    -1
 $EndComp
-Wire Wire Line
-	2600 6250 2700 6250
 Text GLabel 3300 7100 2    50   Output ~ 0
 COLD_SENSE
@@
 L Device:R R?
 U 1 1 60B0B0F6
-P 2450 6250
+P 2400 6400
 AR Path="/60B0B0F6" Ref="R?"  Part="1"
 AR Path="/60AEC464/60B0B0F6" Ref="R208"  Part="1"
-F 0 "R208" V 2350 6350 50  0000 R CNN
-F 1 "7.5K" V 2450 6350 50  0000 R CNN
-F 2 "Resistors_SMD:R_0805_HandSoldering" V 2380 6250 50  0001 C CNN
-F 3 "~" H 2450 6250 50  0001 C CNN
-	1    2450 6250
-	0    -1   -1   0
+F 0 "R208" V 2300 6500 50  0000 R CNN
+F 1 "7.5K" V 2400 6500 50  0000 R CNN
+F 2 "Resistors_SMD:R_0805_HandSoldering" V 2330 6400 50  0001 C CNN
+F 3 "~" H 2400 6400 50  0001 C CNN
+	1    2400 6400
+	1    0    0    -1
 $EndComp
 $Comp
@@
 L power:GND #PWR?
 U 1 1 60A8DFE1
-P 2700 6650
+P 2550 6650
 AR Path="/60A8DFE1" Ref="#PWR?"  Part="1"
 AR Path="/60AEC464/60A8DFE1" Ref="#PWR0215"  Part="1"
-F 0 "#PWR0215" H 2700 6400 50  0001 C CNN
-F 1 "GND" V 2705 6522 50  0000 R CNN
-F 2 "" H 2700 6650 50  0001 C CNN
-F 3 "" H 2700 6650 50  0001 C CNN
-	1    2700 6650
+F 0 "#PWR0215" H 2550 6400 50  0001 C CNN
+F 1 "GND" V 2555 6522 50  0000 R CNN
+F 2 "" H 2550 6650 50  0001 C CNN
+F 3 "" H 2550 6650 50  0001 C CNN
+	1    2550 6650
 	1    0    0    -1
 $EndComp
@@
 	1    0    0    -1
 $EndComp
+Wire Wire Line
+	2300 6250 2400 6250
+Connection ~ 2400 6250
+Wire Wire Line
+	2400 6250 2700 6250
+Wire Wire Line
+	2700 6650 2550 6650
+Wire Wire Line
+	2400 6550 2400 6650
+Wire Wire Line
+	2400 6650 2550 6650
+Connection ~ 2550 6650
 $EndSCHEMATC
