File: kicad/balcony/isense/isense.sch (KiCad schematic (older format))
At the start: 9 parts, among them J1 IN, U1 OPA237NA_250, U2 OPA237NA_250

Commit message: Various schematic fixes
Parts:
- added R7: 100K, Resistor_SMD:R_0805_2012Metric_Pad1.20x1.40mm_HandSolder, symbol Device:R
- added U3: OPA237NA_250, OPA237NA:SOT95P280X145-5N, symbol OPA237NA_250:OPA237NA_250
Connections:
- net +5V: now also U3.5 (V+)
- net GND: now also U3.2 (V-)
- net VIN: now also U3.3 (+IN); no longer R4.2
- net VOUT: now also R7.1; no longer R6.1, U2.1 (OUT)
- new net: R6.1, R7.2, U2.1 (OUT)
- new net: R4.2, U3.1 (OUT), U3.4 (-IN)
Changed lines of the file:
@@
 	7550 1450 7550 2200
-Wire Wire Line
-	7550 2200 7300 2200
 Wire Wire Line
 	6400 1450 5550 1450
@@
 	1    0    0    -1
 $EndComp
-Text Label 5050 2700 2    50   ~ 0
-VIN
 $Comp
 L Connector_Generic:Conn_01x04 J1
@@
 Wire Wire Line
 	1850 2600 1850 2650
-Text Label 7550 2200 0    50   ~ 0
+Text Label 7950 2200 0    50   ~ 0
 VOUT
 Text Label 2150 3400 0    50   ~ 0
 VOUT
+$Comp
+L OPA237NA_250:OPA237NA_250 U3
+U 1 1 6154C66C
+P 3400 3600
+F 0 "U3" H 3400 4170 50  0000 C CNN
+F 1 "OPA237NA_250" H 3400 4079 50  0000 C CNN
+F 2 "OPA237NA:SOT95P280X145-5N" H 3400 3600 50  0001 L BNN
+F 3 "" H 3400 3600 50  0001 L BNN
+	1    3400 3600
+	1    0    0    -1
+$EndComp
+Wire Wire Line
+	2700 3600 2700 4100
+Wire Wire Line
+	4450 3500 4450 4100
+Wire Wire Line
+	2700 4100 4450 4100
+$Comp
+L power:GND #PWR011
+U 1 1 6154C676
+P 4100 3900
+F 0 "#PWR011" H 4100 3650 50  0001 C CNN
+F 1 "GND" H 4105 3727 50  0000 C CNN
+F 2 "" H 4100 3900 50  0001 C CNN
+F 3 "" H 4100 3900 50  0001 C CNN
+	1    4100 3900
+	1    0    0    -1
+$EndComp
+$Comp
+L power:+5V #PWR010
+U 1 1 6154C67C
+P 4100 3300
+F 0 "#PWR010" H 4100 3150 50  0001 C CNN
+F 1 "+5V" H 4115 3473 50  0000 C CNN
+F 2 "" H 4100 3300 50  0001 C CNN
+F 3 "" H 4100 3300 50  0001 C CNN
+	1    4100 3300
+	1    0    0    -1
+$EndComp
+Wire Wire Line
+	4100 3500 4450 3500
+Wire Wire Line
+	2700 3500 2150 3500
+Wire Wire Line
+	5050 2700 4650 2700
+Wire Wire Line
+	4650 2700 4650 3500
+Wire Wire Line
+	4650 3500 4450 3500
+Connection ~ 4450 3500
+$Comp
+L Device:R R7
+U 1 1 615533BA
+P 7800 2200
+F 0 "R7" V 7593 2200 50  0000 C CNN
+F 1 "100K" V 7684 2200 50  0000 C CNN
+F 2 "Resistor_SMD:R_0805_2012Metric_Pad1.20x1.40mm_HandSolder" V 7730 2200 50  0001 C CNN
+F 3 "~" H 7800 2200 50  0001 C CNN
+	1    7800 2200
+	0    1    1    0
+$EndComp
+Wire Wire Line
+	7300 2200 7550 2200
+Connection ~ 7550 2200
+Wire Wire Line
+	7550 2200 7650 2200
 $EndSCHEMATC
